File: mainboard.sch (KiCad schematic (older format))
At the start: 29 parts, among them J1 105017-1001, J2 Conn_01x04_Female, J3 Conn_01x02_Female, J4 Conn_01x09_Female, J5 Conn_01x02_Female, J6 Conn_01x02_Female, J7 Conn_01x04_Female, Q1 AOD4184A, U1 ESP32-WROOM-32E_(16MB), U3 AMS1117-3.3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

Commit message: update volgens feedback
blinkled toegevoegd aan io12
paar grondvias toegevoegd
ingangsontkoppeling ldo
Parts:
- added C10: 10u, Capacitor_SMD:C_0805_2012Metric_Pad1.18x1.45mm_HandSolder, symbol Device:C
- added D1: LED, LED_SMD:LED_0805_2012Metric_Pad1.15x1.40mm_HandSolder, symbol Device:LED
- added R8: TBD, Resistor_SMD:R_0805_2012Metric_Pad1.20x1.40mm_HandSolder, symbol Device:R
Connections:
- net 5V: now also C10.1
- net GND: now also C10.2, D1.1 (K)
- net at U1.14 (IO12): now also R8.2
- new net: D1.2 (A), R8.1
Other:
- moved on the sheet: R6
Changed lines of the file:
@@
 	1    0    0    -1
 $EndComp
-Wire Wire Line
-	9050 1700 9350 1700
 Connection ~ 9350 1700
 Text GLabel 8410 4870 2    50   Input ~ 0
@@
 Text GLabel 4200 1750 2    50   Input ~ 0
 3V3
-Text GLabel 3950 2050 2    50   Input ~ 0
-Mosfet_Trig
 Text Notes 3950 2650 0    50   ~ 0
 PWM\n
@@
 	8450 1100 8450 1400
 Wire Wire Line
-	8450 1400 9050 1400
-Wire Wire Line
-	8200 1500 9050 1500
-Wire Wire Line
-	9050 1500 9050 1700
-Wire Wire Line
-	8200 1700 9050 1700
-Connection ~ 9050 1700
+	8450 1400 8800 1400
+Wire Wire Line
+	8200 1500 8450 1500
 NoConn ~ 8200 1200
 NoConn ~ 8200 1300
@@
 Text GLabel 3950 2150 2    50   Input ~ 0
 PN532_IRQ
-Text GLabel 4550 2250 2    50   Input ~ 0
+Text GLabel 5100 2250 2    50   Input ~ 0
 PN532_RESET
 Text GLabel 3950 3450 2    50   Input ~ 0
@@
 Wire Notes Line
 	470  5320 11210 5320
-Text Notes 5150 2300 0    50   ~ 0
+Text Notes 5750 2250 0    50   ~ 0
 Moet IO5 aan pullup?
 Wire Notes Line
@@
 L Device:R R6
 U 1 1 604E3FBD
-P 4400 2400
-F 0 "R6" H 4500 2350 50  0000 L CNN
-F 1 "10K" H 4500 2450 50  0000 L CNN
-F 2 "Resistor_SMD:R_0805_2012Metric_Pad1.20x1.40mm_HandSolder" V 4330 2400 50  0001 C CNN
-F 3 "~" H 4400 2400 50  0001 C CNN
-	1    4400 2400
-	1    0    0    -1
-$EndComp
-Connection ~ 4400 2250
-Wire Wire Line
-	4400 2250 4550 2250
-Wire Wire Line
-	3950 2250 4400 2250
-Text GLabel 4400 2550 3    50   Input ~ 0
+P 4900 2400
+F 0 "R6" H 5000 2350 50  0000 L CNN
+F 1 "10K" H 5000 2450 50  0000 L CNN
+F 2 "Resistor_SMD:R_0805_2012Metric_Pad1.20x1.40mm_HandSolder" V 4830 2400 50  0001 C CNN
+F 3 "~" H 4900 2400 50  0001 C CNN
+	1    4900 2400
+	1    0    0    -1
+$EndComp
+Connection ~ 4900 2250
+Wire Wire Line
+	4900 2250 5100 2250
+Wire Wire Line
+	3950 2250 4900 2250
+Text GLabel 4900 2550 3    50   Input ~ 0
 3V3
 Wire Wire Line
@@
 	1    0    0    -1
 $EndComp
+Wire Wire Line
+	8200 1700 8450 1700
+Wire Wire Line
+	8450 1500 8450 1700
+Connection ~ 8450 1700
+Wire Wire Line
+	8450 1700 8800 1700
+$Comp
+L Device:C C10
+U 1 1 604E83AF
+P 8800 1550
+F 0 "C10" H 8915 1596 50  0000 L CNN
+F 1 "10u" H 8915 1505 50  0000 L CNN
+F 2 "Capacitor_SMD:C_0805_2012Metric_Pad1.18x1.45mm_HandSolder" H 8838 1400 50  0001 C CNN
+F 3 "~" H 8800 1550 50  0001 C CNN
+	1    8800 1550
+	1    0    0    -1
+$EndComp
+Connection ~ 8800 1400
+Wire Wire Line
+	8800 1400 9050 1400
+Connection ~ 8800 1700
+Wire Wire Line
+	8800 1700 9350 1700
+Text GLabel 3950 2050 2    50   Input ~ 0
+Mosfet_Trig
+$Comp
+L Device:R R8
+U 1 1 604F76FF
+P 4100 2350
+F 0 "R8" V 4100 2250 50  0000 L CNN
+F 1 "TBD" V 4200 2250 50  0000 L CNN
+F 2 "Resistor_SMD:R_0805_2012Metric_Pad1.20x1.40mm_HandSolder" V 4030 2350 50  0001 C CNN
+F 3 "~" H 4100 2350 50  0001 C CNN
+	1    4100 2350
+	0    1    1    0
+$EndComp
+$Comp
+L Device:LED D1
+U 1 1 604F83C9
+P 4400 2350
+F 0 "D1" H 4400 2450 50  0000 C CNN
+F 1 "LED" H 4400 2550 50  0000 C CNN
+F 2 "LED_SMD:LED_0805_2012Metric_Pad1.15x1.40mm_HandSolder" H 4400 2350 50  0001 C CNN
+F 3 "~" H 4400 2350 50  0001 C CNN
+	1    4400 2350
+	-1   0    0    1
+$EndComp
+$Comp
+L power:GND #PWR09
+U 1 1 604F8F1C
+P 4550 2350
+F 0 "#PWR09" H 4550 2100 50  0001 C CNN
+F 1 "GND" V 4555 2222 50  0000 R CNN
+F 2 "" H 4550 2350 50  0001 C CNN
+F 3 "" H 4550 2350 50  0001 C CNN
+	1    4550 2350
+	0    -1   -1   0
+$EndComp
 $EndSCHEMATC
